File: usb-C-breakout.kicad_pcb (KiCad board)
At the start: 2 copper layers, 17.2 x 29.2 mm, 10 parts, among them J1 USB-pins

Commit message: PCB rev to silk
Parts:
- removed the REF** at (105.5, 72.1)
Other:
- board text added: "PCB rev.A"
